File: lcu/motherboard.brd (EAGLE design)
At the start: 117.4 x 83.6 mm, 10 parts

Commit message: Pre finished motherboard
Parts:
- R1: value (none) -> 100R
- moved RELAY 93.6 mm to (50.8, 22.9), turned to 90 degrees
- moved BTN_A 81.3 mm to (26.7, 17.8), turned to 180 degrees
- moved PSU 79.6 mm to (47.0, 72.4), turned to 90 degrees
- moved R1 73.1 mm to (27.9, 34.3), turned to 180 degrees
- moved TMP_SNS 70.0 mm to (36.8, 72.4), turned to 180 degrees
- moved NOTIF 60.3 mm to (26.7, 30.5), turned to 180 degrees
- moved BTN_B 57.7 mm to (26.7, 24.1), turned to 180 degrees
- moved MVM_SNS 42.1 mm to (41.9, 27.9)
- moved DOR_SNS 38.7 mm to (8.89, 27.9)
- moved MCU 10.5 mm to (26.7, 50.8)
Routing:
- net +3V3: track 0.00 -> 193.6 mm, vias 0 -> 8
- net +5V: track 0.00 -> 189.2 mm
- net GND: track 0.00 -> 178.2 mm, vias 0 -> 4
- net D5: track 0.00 -> 81.9 mm, vias 0 -> 2
- net D1: track 0.00 -> 51.6 mm, vias 0 -> 2
- net AD0: track 0.00 -> 43.1 mm, vias 0 -> 2
- net D2: track 0.00 -> 26.3 mm
- net D0: track 0.00 -> 19.1 mm, vias 0 -> 2
- net D3: track 0.00 -> 18.9 mm
- net N$1: track 0.00 -> 6.88 mm
- net D4: track 0.00 -> 6.13 mm
Other:
- board text added: "RELAY"
- board text added: "SWITCH"
