File: lcu/motherboard.brd (EAGLE design)
At the start: 117.4 x 83.6 mm, 10 parts

Commit message: Minor changes in LCU pcb
Other:
- board text added: "PSU"
Changed lines of the file:
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@@
 <setting verticaltext="up"/>
 </settings>
-<grid distance="0.05" unitdist="inch" unit="inch" style="lines" multiple="1" display="no" altdistance="0.025" altunitdist="inch" altunit="inch"/>
+<grid distance="0.05" unitdist="inch" unit="mm" style="lines" multiple="1" display="no" altdistance="0.025" altunitdist="inch" altunit="mm"/>
 <layers>
-<layer number="1" name="Top" color="4" fill="1" visible="no" active="yes"/>
+<layer number="1" name="Top" color="4" fill="1" visible="yes" active="yes"/>
 <layer number="2" name="Route2" color="1" fill="3" visible="no" active="no"/>
 <layer number="3" name="Route3" color="4" fill="3" visible="no" active="no"/>
@@
 <layer number="17" name="Pads" color="2" fill="1" visible="yes" active="yes"/>
 <layer number="18" name="Vias" color="2" fill="1" visible="yes" active="yes"/>
-<layer number="19" name="Unrouted" color="6" fill="1" visible="no" active="yes"/>
+<layer number="19" name="Unrouted" color="6" fill="1" visible="yes" active="yes"/>
 <layer number="20" name="Dimension" color="15" fill="1" visible="yes" active="yes"/>
 <layer number="21" name="tPlace" color="7" fill="1" visible="yes" active="yes"/>
-<layer number="22" name="bPlace" color="7" fill="1" visible="no" active="yes"/>
-<layer number="23" name="tOrigins" color="15" fill="1" visible="no" active="yes"/>
-<layer number="24" name="bOrigins" color="15" fill="1" visible="no" active="yes"/>
-<layer number="25" name="tNames" color="7" fill="1" visible="no" active="yes"/>
-<layer number="26" name="bNames" color="7" fill="1" visible="no" active="yes"/>
-<layer number="27" name="tValues" color="7" fill="1" visible="no" active="yes"/>
-<layer number="28" name="bValues" color="7" fill="1" visible="no" active="yes"/>
-<layer number="29" name="tStop" color="7" fill="3" visible="no" active="yes"/>
-<layer number="30" name="bStop" color="7" fill="6" visible="no" active="yes"/>
-<layer number="31" name="tCream" color="7" fill="4" visible="no" active="yes"/>
-<layer number="32" name="bCream" color="7" fill="5" visible="no" active="yes"/>
-<layer number="33" name="tFinish" color="6" fill="3" visible="no" active="yes"/>
-<layer number="34" name="bFinish" color="6" fill="6" visible="no" active="yes"/>
-<layer number="35" name="tGlue" color="7" fill="4" visible="no" active="yes"/>
-<layer number="36" name="bGlue" color="7" fill="5" visible="no" active="yes"/>
-<layer number="37" name="tTest" color="7" fill="1" visible="no" active="yes"/>
-<layer number="38" name="bTest" color="7" fill="1" visible="no" active="yes"/>
-<layer number="39" name="tKeepout" color="4" fill="11" visible="no" active="yes"/>
-<layer number="40" name="bKeepout" color="1" fill="11" visible="no" active="yes"/>
-<layer number="41" name="tRestrict" color="4" fill="10" visible="no" active="yes"/>
-<layer number="42" name="bRestrict" color="1" fill="10" visible="no" active="yes"/>
-<layer number="43" name="vRestrict" color="2" fill="10" visible="no" active="yes"/>
-<layer number="44" name="Drills" color="7" fill="1" visible="no" active="yes"/>
+<layer number="22" name="bPlace" color="7" fill="1" visible="yes" active="yes"/>
+<layer number="23" name="tOrigins" color="15" fill="1" visible="yes" active="yes"/>
+<layer number="24" name="bOrigins" color="15" fill="1" visible="yes" active="yes"/>
+<layer number="25" name="tNames" color="7" fill="1" visible="yes" active="yes"/>
+<layer number="26" name="bNames" color="7" fill="1" visible="yes" active="yes"/>
+<layer number="27" name="tValues" color="7" fill="1" visible="yes" active="yes"/>
+<layer number="28" name="bValues" color="7" fill="1" visible="yes" active="yes"/>
+<layer number="29" name="tStop" color="7" fill="3" visible="yes" active="yes"/>
+<layer number="30" name="bStop" color="7" fill="6" visible="yes" active="yes"/>
+<layer number="31" name="tCream" color="7" fill="4" visible="yes" active="yes"/>
+<layer number="32" name="bCream" color="7" fill="5" visible="yes" active="yes"/>
+<layer number="33" name="tFinish" color="6" fill="3" visible="yes" active="yes"/>
+<layer number="34" name="bFinish" color="6" fill="6" visible="yes" active="yes"/>
+<layer number="35" name="tGlue" color="7" fill="4" visible="yes" active="yes"/>
+<layer number="36" name="bGlue" color="7" fill="5" visible="yes" active="yes"/>
+<layer number="37" name="tTest" color="7" fill="1" visible="yes" active="yes"/>
+<layer number="38" name="bTest" color="7" fill="1" visible="yes" active="yes"/>
+<layer number="39" name="tKeepout" color="4" fill="11" visible="yes" active="yes"/>
+<layer number="40" name="bKeepout" color="1" fill="11" visible="yes" active="yes"/>
+<layer number="41" name="tRestrict" color="4" fill="10" visible="yes" active="yes"/>
+<layer number="42" name="bRestrict" color="1" fill="10" visible="yes" active="yes"/>
+<layer number="43" name="vRestrict" color="2" fill="10" visible="yes" active="yes"/>
+<layer number="44" name="Drills" color="7" fill="1" visible="yes" active="yes"/>
 <layer number="45" name="Holes" color="7" fill="1" visible="yes" active="yes"/>
-<layer number="46" name="Milling" color="3" fill="1" visible="no" active="yes"/>
+<layer number="46" name="Milling" color="3" fill="1" visible="yes" active="yes"/>
 <layer number="47" name="Measures" color="7" fill="1" visible="yes" active="yes"/>
-<layer number="48" name="Document" color="7" fill="1" visible="no" active="yes"/>
-<layer number="49" name="Reference" color="7" fill="1" visible="no" active="yes"/>
+<layer number="48" name="Document" color="7" fill="1" visible="yes" active="yes"/>
+<layer number="49" name="Reference" color="7" fill="1" visible="yes" active="yes"/>
 <layer number="51" name="tDocu" color="7" fill="1" visible="yes" active="yes"/>
 <layer number="52" name="bDocu" color="7" fill="1" visible="yes" active="yes"/>
@@
 <wire x1="86.22" y1="70.79" x2="86.22" y2="17.79" width="0.4064" layer="21"/>
 <text x="72.39" y="39.37" size="1.778" layer="21" rot="R90">RELAY</text>
-<wire x1="115.58" y1="32.84" x2="115.58" y2="57.84" width="0.4064" layer="21"/>
-<wire x1="115.58" y1="57.84" x2="110.58" y2="62.84" width="0.4064" layer="21"/>
-<wire x1="110.58" y1="62.84" x2="110.58" y2="82.84" width="0.4064" layer="21"/>
-<wire x1="110.58" y1="82.84" x2="86.58" y2="82.84" width="0.4064" layer="21"/>
-<wire x1="86.58" y1="82.84" x2="86.58" y2="62.84" width="0.4064" layer="21"/>
-<wire x1="86.58" y1="62.84" x2="93.58" y2="62.84" width="0.4064" layer="21"/>
-<wire x1="93.58" y1="62.84" x2="93.58" y2="32.84" width="0.4064" layer="21"/>
-<wire x1="93.58" y1="32.84" x2="115.58" y2="32.84" width="0.4064" layer="21"/>
 <wire x1="89.99" y1="31.265" x2="116.99" y2="31.265" width="0.4064" layer="21"/>
 <wire x1="116.99" y1="31.265" x2="116.99" y2="4.265" width="0.4064" layer="21"/>
@@
 <wire x1="89.99" y1="4.265" x2="89.99" y2="31.265" width="0.4064" layer="21"/>
 <text x="97.99" y="18.265" size="1.778" layer="21">SWITCH</text>
+<wire x1="87.145" y1="77.965" x2="87.145" y2="52.965" width="0.4064" layer="21"/>
+<wire x1="87.145" y1="77.965" x2="107.145" y2="77.965" width="0.4064" layer="21"/>
+<wire x1="107.145" y1="77.965" x2="107.145" y2="52.965" width="0.4064" layer="21"/>
+<wire x1="107.145" y1="52.965" x2="115.145" y2="52.965" width="0.4064" layer="21"/>
+<wire x1="115.145" y1="52.965" x2="115.145" y2="32.965" width="0.4064" layer="21"/>
+<wire x1="115.145" y1="32.965" x2="91.145" y2="32.965" width="0.4064" layer="21"/>
+<wire x1="91.145" y1="32.965" x2="91.145" y2="50.965" width="0.4064" layer="21"/>
+<wire x1="91.145" y1="50.965" x2="87.145" y2="52.965" width="0.4064" layer="21"/>
+<text x="103.505" y="51.435" size="1.778" layer="21" rot="R180">PSU</text>
 </plain>
 <attributes>
@@
 <param name="rvMicroViaOuter" value="0.25"/>
 <param name="rvMicroViaInner" value="0.25"/>
-<param name="rlMinPadTop" value="17mil"/>
+<param name="rlMinPadTop" value="20mil"/>
 <param name="rlMaxPadTop" value="20mil"/>
 <param name="rlMinPadInner" value="10mil"/>
@@
 <param name="rlMinPadBottom" value="10mil"/>
 <param name="rlMaxPadBottom" value="20mil"/>
-<param name="rlMinViaOuter" value="14mil"/>
+<param name="rlMinViaOuter" value="20mil"/>
 <param name="rlMaxViaOuter" value="20mil"/>
 <param name="rlMinViaInner" value="8mil"/>
@@
 <wire x1="6.7" y1="6.85" x2="58.7" y2="6.85" width="0" layer="19" extent="1-1"/>
 </signal>
+<signal name="N$3">
+<via x="60.96" y="67.31" extent="1-16" drill="3"/>
+</signal>
+<signal name="N$4">
+<via x="82.55" y="67.31" extent="1-16" drill="3"/>
+</signal>
+<signal name="N$5">
+<via x="82.55" y="21.59" extent="1-16" drill="3"/>
+</signal>
+<signal name="N$6">
+<via x="60.96" y="21.59" extent="1-16" drill="3"/>
+</signal>
 </signals>
