File: lcu/motherboard.sch (EAGLE design)
At the start: 2 parts

Commit message: Casing in eagle
Parts:
- added BTN_A, BTN_B, NOTIF: (no value), pinhead:PINHD-1X2
- added DOR_SNS, MVM_SNS, TMP_SNS: (no value), pinhead:PINHD-2X2
- added R1: (no value), rcl:R-EU_0204/7
- added RELAY: (no value), pinhead:PINHD-1X3
- renumbered JP1 to PSU, U$1 to MCU
Connections:
- removed net VCC: MCU.VIN, PSU.2
- new net +5V: DOR_SNS.1, MCU.VIN, MVM_SNS.1, PSU.2, RELAY.1, TMP_SNS.1
- new net AD0: MCU.AD0, TMP_SNS.3
- new net D0: MCU.D0, MVM_SNS.3
- new net D1: DOR_SNS.3, MCU.D1
- new net D2: BTN_A.1, MCU.D2
- new net D3: BTN_B.1, MCU.D3
- new net D4: MCU.D4, R1.1
- new net D5: MCU.D5, RELAY.2
- new net N$1: NOTIF.1, R1.2
- net +3V3: now also DOR_SNS.2, MVM_SNS.2, TMP_SNS.2
- net GND: now also BTN_A.2, BTN_B.2, DOR_SNS.4, MVM_SNS.4, NOTIF.2, RELAY.3, TMP_SNS.4
Other:
- note added: "Input/Output"

Commit message: Pre finished motherboard
Parts:
- R1: value (none) -> 100R
Changed lines of the file:
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@@
 <part name="GND9" library="supply1" deviceset="GND" device=""/>
 <part name="GND10" library="supply1" deviceset="GND" device=""/>
-<part name="R1" library="rcl" deviceset="R-EU_" device="0204/7"/>
+<part name="R1" library="rcl" deviceset="R-EU_" device="0204/7" value="100R"/>
 </parts>
 <sheets>

Commit message: Minor changes in LCU pcb
Other:
- note added: "WIFI MCU"
- moved on the sheet: PSU
Changed lines of the file:
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@@
 <sheet>
 <plain>
-<wire x1="-66.04" y1="81.28" x2="-66.04" y2="53.34" width="0.1524" layer="97" style="shortdash"/>
-<wire x1="-66.04" y1="53.34" x2="-20.32" y2="53.34" width="0.1524" layer="97" style="shortdash"/>
-<wire x1="-20.32" y1="53.34" x2="-20.32" y2="81.28" width="0.1524" layer="97" style="shortdash"/>
-<wire x1="-20.32" y1="81.28" x2="-66.04" y2="81.28" width="0.1524" layer="97" style="shortdash"/>
-<text x="-63.5" y="76.2" size="2.54" layer="97">PSU Connector</text>
+<wire x1="-63.5" y1="93.98" x2="-63.5" y2="66.04" width="0.1524" layer="97" style="shortdash"/>
+<wire x1="-63.5" y1="66.04" x2="-17.78" y2="66.04" width="0.1524" layer="97" style="shortdash"/>
+<wire x1="-17.78" y1="66.04" x2="-17.78" y2="93.98" width="0.1524" layer="97" style="shortdash"/>
+<wire x1="-17.78" y1="93.98" x2="-63.5" y2="93.98" width="0.1524" layer="97" style="shortdash"/>
+<text x="-60.96" y="88.9" size="2.54" layer="97">PSU Connector</text>
 <wire x1="81.28" y1="93.98" x2="81.28" y2="0" width="0.1524" layer="97" style="shortdash"/>
 <wire x1="81.28" y1="0" x2="190.5" y2="0" width="0.1524" layer="97" style="shortdash"/>
@@
 <wire x1="190.5" y1="93.98" x2="81.28" y2="93.98" width="0.1524" layer="97" style="shortdash"/>
 <text x="129.54" y="88.9" size="2.54" layer="97">Input/Output</text>
+<wire x1="-15.24" y1="93.98" x2="-15.24" y2="0" width="0.1524" layer="97" style="shortdash"/>
+<wire x1="-15.24" y1="0" x2="71.12" y2="0" width="0.1524" layer="97" style="shortdash"/>
+<wire x1="71.12" y1="0" x2="71.12" y2="93.98" width="0.1524" layer="97" style="shortdash"/>
+<wire x1="71.12" y1="93.98" x2="-15.24" y2="93.98" width="0.1524" layer="97" style="shortdash"/>
+<text x="17.78" y="83.82" size="2.54" layer="97">WIFI MCU</text>
 </plain>
 <instances>
@@
 <attribute name="VALUE" x="55.88" y="73.66" size="1.778" layer="96"/>
 </instance>
-<instance part="PSU" gate="G$1" x="-45.72" y="68.58" rot="R180"/>
-<instance part="GND3" gate="1" x="-35.56" y="60.96"/>
+<instance part="PSU" gate="G$1" x="-43.18" y="81.28" rot="R180"/>
+<instance part="GND3" gate="1" x="-33.02" y="73.66"/>
 <instance part="MVM_SNS" gate="A" x="157.48" y="43.18"/>
 <instance part="TMP_SNS" gate="A" x="157.48" y="63.5"/>
@@
 <attribute name="VALUE" x="-6.985" y="36.195" size="1.778" layer="96"/>
 </instance>
-<instance part="SUPPLY1" gate="+5V" x="-35.56" y="73.66"/>
+<instance part="SUPPLY1" gate="+5V" x="-33.02" y="86.36"/>
 <instance part="SUPPLY2" gate="+5V" x="111.76" y="22.86" smashed="yes">
 <attribute name="VALUE" x="104.775" y="23.495" size="1.778" layer="96"/>
@@
 <segment>
 <pinref part="PSU" gate="G$1" pin="1"/>
-<wire x1="-43.18" y1="66.04" x2="-35.56" y2="66.04" width="0.1524" layer="91"/>
+<wire x1="-40.64" y1="78.74" x2="-33.02" y2="78.74" width="0.1524" layer="91"/>
 <pinref part="GND3" gate="1" pin="GND"/>
-<wire x1="-35.56" y1="66.04" x2="-35.56" y2="63.5" width="0.1524" layer="91"/>
+<wire x1="-33.02" y1="78.74" x2="-33.02" y2="76.2" width="0.1524" layer="91"/>
 </segment>
 <segment>
@@
 <segment>
 <pinref part="PSU" gate="G$1" pin="2"/>
-<wire x1="-43.18" y1="68.58" x2="-35.56" y2="68.58" width="0.1524" layer="91"/>
-<wire x1="-35.56" y1="68.58" x2="-35.56" y2="71.12" width="0.1524" layer="91"/>
+<wire x1="-40.64" y1="81.28" x2="-33.02" y2="81.28" width="0.1524" layer="91"/>
+<wire x1="-33.02" y1="81.28" x2="-33.02" y2="83.82" width="0.1524" layer="91"/>
 <pinref part="SUPPLY1" gate="+5V" pin="+5V"/>
 </segment>
