File: lcu/motherboard/motherboard.brd (EAGLE design)
At the start: 160 x 100 mm, 10 parts

Commit message: New motherboard and IOBoard
Parts:
- removed DOR_SNS, MVM_SNS, TMP_SNS: (no value), pinhead:2X02
- added IOBRD_POW: (no value), pinhead:2X02
- added IO_BRD: (no value), pinhead:1X09
- R1: value (none) -> 100R
- moved R1 102.9 mm to (53.3, 17.8), turned to 90 degrees
- moved BTN_A 97.4 mm to (48.3, 31.8), turned to 90 degrees
- moved NOTIF 86.7 mm to (48.3, 15.2), turned to 90 degrees
- moved RELAY 86.4 mm to (48.3, 55.9), turned to 270 degrees
- moved BTN_B 76.2 mm to (48.3, 22.9), turned to 270 degrees
- moved PSU 75.8 mm to (43.2, 72.4), turned to 90 degrees
- moved MCU 58.6 mm to (29.2, 43.2), turned to 180 degrees
Connections:
- new net D6: IO_BRD.6, MCU.D6
- new net D7: IO_BRD.7, MCU.D7
- new net D8: MCU.D8, RELAY.2
- new net NC: IO_BRD.8
- new net SD2: BTN_A.1, MCU.SD2
- new net SD3: BTN_B.1, MCU.SD3
- net +3V3: now also IOBRD_POW.2, R1.2; no longer DOR_SNS.2, MVM_SNS.2, TMP_SNS.2
- net +5V: now also IOBRD_POW.1; no longer DOR_SNS.1, MVM_SNS.1, TMP_SNS.1
- net AD0: now also IO_BRD.9; no longer TMP_SNS.3
- net D0: now also NOTIF.2; no longer MVM_SNS.3
- net D1: now also IO_BRD.1; no longer DOR_SNS.3
- net D2: now also IO_BRD.2; no longer BTN_A.1
- net D3: now also IO_BRD.3; no longer BTN_B.1
- net D4: now also IO_BRD.4; no longer R1.1
- net D5: now also IO_BRD.5; no longer RELAY.2
- net GND: now also IOBRD_POW.4; no longer DOR_SNS.4, MVM_SNS.4, NOTIF.2, TMP_SNS.4
- net N$1: now also R1.1; no longer R1.2
Routing:
- net GND: track 0.00 -> 225.9 mm
- net +3V3: track 0.00 -> 98.5 mm, vias 0 -> 2
- net +5V: track 0.00 -> 80.1 mm, vias 0 -> 2
- net AD0: track 0.00 -> 74.2 mm, vias 0 -> 2
- net D0: track 0.00 -> 34.2 mm
- net D8: track 0.00 -> 32.6 mm, vias 0 -> 2
- net D4: track 0.00 -> 13.5 mm
- net SD3: track 0.00 -> 12.8 mm
- net D2: track 0.00 -> 12.8 mm
- net D1: track 0.00 -> 12.8 mm
- net D3: track 0.00 -> 12.8 mm
- net D7: track 0.00 -> 10.7 mm
- net D6: track 0.00 -> 10.7 mm
- net D5: track 0.00 -> 10.7 mm
- net SD2: track 0.00 -> 10.5 mm
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Other:
- board size 160 x 100 mm -> 117.4 x 83.6 mm
- board text added: "PSU"
- board text added: "RELAY"
- board text added: "SWITCH"
